File: ecomodbus_hardware/PCB/ecoBeat_3.kicad_pcb (KiCad board)
At the start: 2 copper layers, 120.2 x 129.4 mm, 24 parts, among them IC1 ATTINY85-P, J1 RJ45, P1 CONN_01X06, P3 CONN_01X02, SW1 SW_PUSH, SW2 SW_PUSH, U1 ESP-12E, U2 AP1117D33

Commit message: hardware intermiedio
Parts:
- removed C3, C4: 10uF, Capacitors_ThroughHole:C_Radial_D5_L11_P2
- removed D1, D2, D3: LED, LEDs:LED-3MM
- removed D4: D, Diodes_ThroughHole:Diode_DO-35_SOD27_Horizontal_RM10
- removed IC1: ATTINY85-P, Housings_DIP:DIP-8_W7.62mm
- removed J1: RJ45, Connect:RJ45_8
- removed P1: CONN_01X06, Pin_Headers:Pin_Header_Straight_1x06
- removed P3: CONN_01X02, Connect:bornier2
- removed SW1, SW2: SW_PUSH, Buttons_Switches_ThroughHole:SW_PUSH_SMALL
- added C2: 10uF, Capacitors_THT:CP_Radial_D5.0mm_P2.00mm, F.Cu at (117.1, 84.8)
- added R10: 120, Resistors_THT:R_Axial_DIN0207_L6.3mm_D2.5mm_P10.16mm_Horizontal, F.Cu at (88.6, 120.1)
- C1: value 100nF -> 10nF; footprint Capacitors_ThroughHole:C_Disc_D3_P2.5 -> Capacitors_THT:C_Disc_D5.0mm_W2.5mm_P5.00mm
- R1, R2, R3: value 10k -> 10K; footprint Resistors_ThroughHole:Resistor_Horizontal_RM7mm -> Resistors_THT:R_Axial_DIN0207_L6.3mm_D2.5mm_P10.16mm_Horizontal
- R4: value 6.8k -> 10K; footprint Resistors_ThroughHole:Resistor_Horizontal_RM7mm -> Resistors_THT:R_Axial_DIN0207_L6.3mm_D2.5mm_P10.16mm_Horizontal
- R5: value 12k -> 20K; footprint Resistors_ThroughHole:Resistor_Horizontal_RM7mm -> Resistors_THT:R_Axial_DIN0207_L6.3mm_D2.5mm_P10.16mm_Horizontal
- R6, R7, R8: footprint Resistors_ThroughHole:Resistor_Horizontal_RM7mm -> Resistors_THT:R_Axial_DIN0207_L6.3mm_D2.5mm_P10.16mm_Horizontal
- R9: value 10k -> 20K; footprint Resistors_ThroughHole:Resistor_Horizontal_RM7mm -> Resistors_THT:R_Axial_DIN0207_L6.3mm_D2.5mm_P10.16mm_Horizontal
- U1: value ESP-12E -> WeMos_mini; footprint ESP8266:ESP-07v2 -> wemos_d1_mini:D1_mini_board
- U2: value AP1117D33 -> ACDC-5V; footprint TO_SOT_Packages_SMD:SOT-223 -> ac-dc_VTX:vigortronix; moved to F.Cu
- moved R4 105.0 mm to (87.9, 147.3), turned to 0 degrees
- moved R9 99.6 mm to (67.3, 85.3), turned to 0 degrees
- moved R7 73.3 mm to (128.0, 152.7), turned to 0 degrees
- moved R6 71.4 mm to (109.0, 153.4), turned to 0 degrees
- moved R5 65.8 mm to (157.0, 139.4), turned to 0 degrees
- moved R1 59.9 mm to (127.0, 70.1)
- moved U2 51.5 mm to (113.8, 124.7), turned to 90 degrees
- moved R2 48.0 mm to (176.5, 144.3), turned to 0 degrees
- moved R8 43.1 mm to (158.0, 152.9), turned to 0 degrees
- moved C1 40.9 mm to (119.6, 89.7)
- moved U1 31.5 mm to (120.4, 65.0)
- moved R3 31.3 mm to (133.6, 145.5)
Connections:
- C1 pad 1: VCC -> /5.0V
- C1 pad 2: GND -> Net-(C1-Pad2)
- R1 pad 1: Net-(IC1-Pad7) -> Net-(R1-Pad1)
- R1 pad 2: GND -> /5.0V
- R2 pad 1: VCC -> Net-(R2-Pad1)
- R2 pad 2: ESPRST -> /5.0V
- R3 pad 1: VCC -> Net-(R3-Pad1)
- R3 pad 2: RSTTINY -> /5.0V
- R4 pad 1: Net-(P1-Pad3) -> Net-(R4-Pad1)
- R4 pad 2: RXD -> /5.0V
- R5 pad 1: GND -> Net-(J2-Pad1)
- R5 pad 2: RXD -> /5.0V
- R9 pad 1: Net-(R9-Pad1) -> GND
- R9 pad 2: VCC -> Net-(J2-Pad2)
- U1 pad 1: ESPRST -> /5.0V
- U1 pad 10: GND -> Net-(U1-Pad10)
- U1 pad 11: VCC -> Net-(U1-Pad11)
- U1 pad 12: Net-(R9-Pad1) -> Net-(R4-Pad1)
- U1 pad 13: RX1 -> Net-(R3-Pad1)
- U1 pad 14: TX1 -> Net-(R2-Pad1)
- U1 pad 15: RXD -> Net-(R1-Pad1)
- U1 pad 16: TXD -> Net-(U1-Pad16)
- U1 pad 2: VCC -> GND
- U1 pad 3: VCC -> /L1
- U1 pad 4: L2 -> /L2
- U1 pad 5: RSTTINY -> Net-(U1-Pad5)
- U1 pad 6: INT1 -> Net-(U1-Pad6)
- U1 pad 8: VCC -> Net-(U1-Pad8)
- U1 pad 9: GND -> Net-(U1-Pad9)
- U2 pad 1: GND -> Net-(F1-Pad2)
- U2 pad 2: VCC -> Net-(J1-Pad1)
- U2 pad 3: Net-(C3-Pad1) -> Net-(C1-Pad2)
Routing:
- net VCC: track 141.3 -> 0.00 mm
- net ESPRST: track 72.7 -> 0.00 mm
- net RSTTINY: track 48.7 -> 0.00 mm
- net RX1: track 41.2 -> 0.00 mm
- net TX1: track 40.6 -> 0.00 mm
- net L2: track 37.9 -> 0.00 mm
- net INT1: track 35.2 -> 0.00 mm
- net GND: track 32.1 -> 0.00 mm
- net TXD: track 27.1 -> 0.00 mm
- net Net-(R9-Pad1): track 22.5 -> 0.00 mm
- net L1: track 22.2 -> 0.00 mm
- net Net-(IC1-Pad7): track 20.3 -> 0.00 mm
- net RXD: track 15.3 -> 0.00 mm
- net Net-(C3-Pad1): track 14.3 -> 0.00 mm
- net Net-(D1-Pad1): track 13.1 -> 0.00 mm
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Other:
- board size 120.2 x 129.4 mm -> 30.9 x 86 mm
- board text removed: "RESET"
