File: ecomodbus_hardware/PCB/ecoBeat_3.kicad_pcb (KiCad board)
At the start: 2 copper layers, 30.9 x 86 mm, 14 parts, among them U1 WeMos_mini, U2 ACDC-5V

Commit message: primera version PCB para pruebas
Parts:
- removed R7: 220, Resistors_THT:R_Axial_DIN0207_L6.3mm_D2.5mm_P10.16mm_Horizontal
- added D1: LED, LEDs:LED-3MM, F.Cu at (127.1, 85.9)
- added D3: LED, LEDs:LED-3MM, F.Cu at (132.5, 86.1)
- added F1: Fuse, fuse:Fuse_Horizontal_RM10mm, F.Cu at (132.7, 120.1)
- added J1: AC_input, Connect:bornier2, F.Cu at (128.3, 128.3)
- added J2: Conn_MODBUS, Connect:bornier3, F.Cu at (114.3, 128.3)
- added J3: Test_5V, Wire_Pads:SolderWirePad_single_0-8mmDrill, F.Cu at (119.5, 83.3)
- added P1: CONN_VCC, Pin_Headers:Pin_Header_Straight_1x08, F.Cu at (131.7, 55.1)
- added P2: CONN_DATOS, Pin_Headers:Pin_Header_Straight_1x08, F.Cu at (108.9, 72.9)
- added U3: MAX_485, SMD_Packages:SOIC-8-N, F.Cu at (117.1, 63.7)
- C1: footprint Capacitors_THT:C_Disc_D5.0mm_W2.5mm_P5.00mm -> Capacitors_SMD:C_1206_HandSoldering
- C2: footprint Capacitors_THT:CP_Radial_D5.0mm_P2.00mm -> Capacitors_SMD:C_1206_HandSoldering
- R1, R10, R2, R3, R4, R5, R6, R8, R9: footprint Resistors_THT:R_Axial_DIN0207_L6.3mm_D2.5mm_P10.16mm_Horizontal -> Resistors_SMD:R_1206
- moved R2 107.7 mm to (115.5, 55.5), turned to 90 degrees
- moved R4 97.8 mm to (121.5, 55.5), turned to 90 degrees
- moved R3 91.3 mm to (118.5, 55.5), turned to 90 degrees
- moved R8 80.2 mm to (131.7, 77.1), turned to 90 degrees
- moved R6 78.6 mm to (127.9, 77.1), turned to 90 degrees
- moved R5 73.1 mm to (118.7, 77.1), turned to 270 degrees
- moved U1 67.6 mm to (187.9, 61.3)
- moved R10 58.4 mm to (122.5, 72.5)
- moved R9 56.4 mm to (123.1, 77.1), turned to 90 degrees
- moved R1 20.6 mm to (112.5, 55.5), turned to 90 degrees
- moved C1 6.51 mm to (114.3, 85.9)
- moved U2 5.67 mm to (111.1, 119.7)
- moved C2 3.17 mm to (114.3, 83.3)
Connections:
- net /L2 renamed Net-(U1-Pad4)
- C1 pad 2: Net-(C1-Pad2) -> GND
- C2 pad 2: Net-(C1-Pad2) -> GND
- R1 pad 1: Net-(R1-Pad1) -> Net-(P2-Pad5)
- R2 pad 1: Net-(R2-Pad1) -> Net-(P2-Pad4)
- R3 pad 1: Net-(R3-Pad1) -> Net-(P2-Pad3)
- R4 pad 1: Net-(R4-Pad1) -> Net-(P2-Pad2)
- R6 pad 1: GND -> Net-(D1-Pad2)
- R6 pad 2: Net-(D1-Pad1) -> /L1
- R8 pad 1: GND -> Net-(D3-Pad2)
- R8 pad 2: Net-(D3-Pad1) -> /5.0V
- U1 pad 1: /5.0V -> Net-(U1-Pad1)
- U1 pad 12: Net-(R4-Pad1) -> Net-(U1-Pad12)
- U1 pad 13: Net-(R3-Pad1) -> Net-(U1-Pad13)
- U1 pad 14: Net-(R2-Pad1) -> Net-(U1-Pad14)
- U1 pad 15: Net-(R1-Pad1) -> Net-(U1-Pad15)
- U1 pad 2: GND -> Net-(U1-Pad2)
- U1 pad 3: /L1 -> Net-(U1-Pad3)
- U2 pad 3: Net-(C1-Pad2) -> GND
Routing:
- net GND: track 0.00 -> 129.0 mm, vias 0 -> 1
- net /5.0V: track 0.00 -> 113.2 mm, vias 0 -> 1
- net Net-(J2-Pad2): track 0.00 -> 87.5 mm
- net Net-(J2-Pad1): track 0.00 -> 78.7 mm
- net Net-(J1-Pad1): track 0.00 -> 20.3 mm
- net Net-(P2-Pad2): track 0.00 -> 20.2 mm
- net Net-(P2-Pad3): track 0.00 -> 16.8 mm
- net Net-(P2-Pad4): track 0.00 -> 14.0 mm
- net Net-(F1-Pad2): track 0.00 -> 14.0 mm
- net /L1: track 0.00 -> 13.5 mm
- net Net-(P2-Pad5): track 0.00 -> 10.9 mm
- net Net-(F1-Pad1): track 0.00 -> 8.94 mm
- net Net-(D3-Pad2): track 0.00 -> 5.34 mm
- net Net-(D1-Pad2): track 0.00 -> 5.14 mm
Other:
- rule trace_min: 0.4 -> 0.1
- board text removed: "FLASH"

Commit message: pdb 2
Parts:
- removed J1: AC_input, Connect:bornier2
- removed J2: Conn_MODBUS, Connect:bornier3
- added J3: L1, Wire_Pads:SolderWirePad_single_0-8mmDrill, F.Cu at (123.2, 55.4)
- added J3: L1, Wire_Pads:SolderWirePad_single_0-8mmDrill, F.Cu at (124.5, 70.4)
- added J3: L1, Wire_Pads:SolderWirePad_single_0-8mmDrill, F.Cu at (129.5, 76.2)
- added J3: L1, Wire_Pads:SolderWirePad_single_0-8mmDrill, F.Cu at (108.5, 75.9)
- added J3: GND, Wire_Pads:SolderWirePad_single_0-8mmDrill, F.Cu at (109.0, 103.4)
- added P3: CONN_01X06, Connect:bornier6, F.Cu at (120.3, 127.3)
- U1, U2: moved to B.Cu
- moved F1 24.8 mm to (108.0, 121.3)
- moved P2 23.2 mm to (132.1, 72.4)
- moved P1 22.5 mm to (109.2, 54.6)
- moved U2 19.1 mm to (130.2, 119.4)
- moved J3 18.1 mm to (109.0, 98.0)
- moved R1 16.1 mm to (128.0, 59.7)
- moved R2 10.8 mm to (125.5, 59.7)
- moved U1 9.28 mm to (179.1, 64.1), turned to 180 degrees
- moved C1 8.83 mm to (111.8, 77.5), turned to 270 degrees
- moved U3 7.71 mm to (124.5, 66.0), turned to 90 degrees
- moved R10 7.69 mm to (115.6, 69.2)
- moved R3 6.27 mm to (123.2, 59.7)
- moved R4 4.26 mm to (120.7, 59.7)
- moved R5 2.53 mm to (116.2, 77.5)
- moved D3 1.72 mm to (132.1, 84.5)
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Connections:
- F1 pad 1: Net-(F1-Pad1) -> N_IN
- U2 pad 2: Net-(J1-Pad1) -> L_IN
- U3 pad 1: Net-(P2-Pad5) -> Net-(P2-Pad2)
- U3 pad 2: Net-(P2-Pad4) -> Net-(P2-Pad3)
- U3 pad 3: Net-(P2-Pad3) -> Net-(P2-Pad4)
- U3 pad 4: Net-(P2-Pad2) -> Net-(P2-Pad5)
Routing:
- net GND: track 129.0 -> 7.71 mm, vias 1 -> 0
- net /L1: track 13.5 -> 37.7 mm
- net L_IN: track 0.00 -> 22.2 mm
- net Net-(J1-Pad1): track 20.3 -> 0.00 mm
- net Net-(F1-Pad1): track 8.94 -> 0.00 mm
- net Net-(P3-Pad2): track 78.7 -> 86.1 mm
- net N_IN: track 0.00 -> 6.14 mm
- net /5.0V: track 113.2 -> 118.5 mm, vias 1 -> 0
- net Net-(P3-Pad1): track 87.5 -> 83.1 mm
- net Net-(P2-Pad3): track 16.8 -> 12.8 mm
- net Net-(P2-Pad4): track 14.0 -> 10.6 mm
- net Net-(P2-Pad2): track 20.2 -> 17.0 mm
- net Net-(P2-Pad5): track 10.9 -> 7.68 mm
- net Net-(D3-Pad2): track 5.34 -> 3.00 mm
- net Net-(D1-Pad2): track 5.14 -> 3.00 mm
- added copper zone on F.Cu, net GND
- removed copper zone on B.Cu, net GND
