File: ecomodbus_hardware/PCB/ecoBeat_3.kicad_pcb (KiCad board)
At the start: 2 copper layers, 30.9 x 86 mm, 22 parts, among them J1 AC_input, J2 Conn_MODBUS, J3 Test_5V, P1 CONN_VCC, P2 CONN_DATOS, U1 WeMos_mini, U2 ACDC-5V, U3 MAX_485

Commit message: primera version para probar
Parts:
- moved R1 17.8 mm to (126.3, 66.7), turned to 270 degrees
- moved U1 11.9 mm to (179.3, 69.5)
- moved R2 11.3 mm to (114.1, 66.7), turned to 270 degrees
- moved R4 5.00 mm to (126.3, 56.9)
- moved R3 4.62 mm to (114.1, 56.9)
- moved U3 3.26 mm to (120.3, 63.1), turned to 180 degrees
- moved D3 0.45 mm to (132.1, 85.9)
Connections:
- net Net-(P2-Pad4) renamed /receiver
- P1 pad 1: Net-(P1-Pad1) -> /tx_wemos
- P1 pad 2: Net-(P1-Pad2) -> /rx_wemos
- P2 pad 5: Net-(P2-Pad5) -> /driver
- R1 pad 1: Net-(P2-Pad5) -> /rx_wemos
- R3 pad 1: Net-(P2-Pad3) -> /driver
- R4 pad 1: Net-(P2-Pad2) -> /tx_wemos
- U3 pad 1: Net-(P2-Pad5) -> /rx_wemos
- U3 pad 3: Net-(P2-Pad3) -> /driver
- U3 pad 4: Net-(P2-Pad2) -> /tx_wemos
Routing:
- net Net-(P2-Pad2): track 20.2 -> 0.00 mm
- net /tx_wemos: track 0.00 -> 17.3 mm
- net /driver: track 0.00 -> 16.8 mm
- net /rx_wemos: track 0.00 -> 16.0 mm
- net Net-(P2-Pad3): track 16.8 -> 0.88 mm
- net Net-(P2-Pad5): track 10.9 -> 0.00 mm
- net Net-(J2-Pad2): track 87.5 -> 80.6 mm
- net /5.0V: track 113.2 -> 109.0 mm, vias 1 -> 5
- net Net-(J2-Pad1): track 78.7 -> 74.6 mm
- net /receiver: track 14.0 -> 15.9 mm
- net GND: track 129.0 -> 127.6 mm
- net /L1: track 13.5 -> 12.5 mm

Commit message: version de fabricacion
Parts:
- removed U1: WeMos_mini, wemos_d1_mini:D1_mini_board
