File: ecomodbus_hardware/PCB/ecoBeat_3.sch (KiCad schematic (older format))
At the start: 26 parts, among them IC1 ATTINY85-P, J1 RJ45, P1 CONN_01X06, P3 CONN_01X02, SW2 SW_PUSH, U1 ESP-12E, U2 AP1117D33

Commit message: hardware intermiedio
Parts:
- removed C1: 100nF, Discret:CP36V, symbol CP
- removed C3, C4: 10uF, Capacitors_ThroughHole:C_Disc_D3_P2.5, symbol C
- removed D?: D, symbol D
- removed IC1: ATTINY85-P, Housings_DIP:DIP-8_W7.62mm, symbol ATTINY85-P-RESCUE-ecoBeat_3
- removed J1: RJ45, Connect:RJ45_8, symbol RJ45
- removed P1: CONN_01X06, Pin_Headers:Pin_Header_Straight_1x06, symbol CONN_01X06
- removed P3: CONN_01X02, Connect:bornier2, symbol CONN_01X02
- removed SW2: SW_PUSH, Buttons_Switches_ThroughHole:SW_PUSH_SMALL, symbol SW_PUSH
- removed U1: ESP-12E, ESP8266:ESP-12E, symbol ESP-12E
- removed U2: AP1117D33, TO_SOT_Packages_SMD:SOT-223, symbol AP1117D33
- removed U?: MAX_485, SO-8, symbol MAX_485
- added C1: 10nF, Capacitors_THT:C_Disc_D5.0mm_W2.5mm_P5.00mm, symbol C
- added C2: 10uF, Capacitors_THT:CP_Radial_D5.0mm_P2.00mm, symbol CP
- added F1: Fuse, symbol Fuse_Small
- added J1: AC_input, symbol Conn_01x02
- added J2: Conn_MODBUS, symbol Conn_01x03
- added J3: Test_5V, symbol TEST_1P
- added U2: ACDC-5V, ac-dc_VTX:vigortronix, symbol ACDC-5V
- added U3: MAX_485, SMD_Packages:SOIC-8-N, symbol MAX_485
- R1, R2, R3: value 10k -> 10K; footprint Resistors_ThroughHole:Resistor_Horizontal_RM7mm -> Resistors_THT:R_Axial_DIN0207_L6.3mm_D2.5mm_P10.16mm_Horizontal
- R10: value 10k -> 120; footprint Resistors_ThroughHole:Resistor_Horizontal_RM7mm -> Resistors_THT:R_Axial_DIN0207_L6.3mm_D2.5mm_P10.16mm_Horizontal
- R4: value 6.8k -> 10K; footprint Resistors_ThroughHole:Resistor_Horizontal_RM7mm -> Resistors_THT:R_Axial_DIN0207_L6.3mm_D2.5mm_P10.16mm_Horizontal
- R5: value 12k -> 20K; footprint Resistors_ThroughHole:Resistor_Horizontal_RM7mm -> Resistors_THT:R_Axial_DIN0207_L6.3mm_D2.5mm_P10.16mm_Horizontal
- R6, R7, R8: footprint Resistors_ThroughHole:Resistor_Horizontal_RM7mm -> Resistors_THT:R_Axial_DIN0207_L6.3mm_D2.5mm_P10.16mm_Horizontal
- R9: value 10k -> 20K; footprint Resistors_ThroughHole:Resistor_Horizontal_RM7mm -> Resistors_THT:R_Axial_DIN0207_L6.3mm_D2.5mm_P10.16mm_Horizontal
- U1: renamed from U?; footprint (none) -> wemos_d1_mini:D1_mini_board
Connections:
- net labels added: 5.0V
- net labels removed: 3.3, ESPRST, INT1, RSTTINY, RX1, RXD, TX1, TXD
- wire segments 92 -> 55
- no-connect marks 26 -> 8
Other:
- moved on the sheet: D1, D2, D3, R6, R7, R8, U1

Commit message: primera version PCB para pruebas
Parts:
- removed D2: LED, LEDs:LED-3MM, symbol LED
- removed R7: 220, Resistors_THT:R_Axial_DIN0207_L6.3mm_D2.5mm_P10.16mm_Horizontal, symbol R
- added P1: CONN_VCC, Pin_Headers:Pin_Header_Straight_1x08, symbol CONN_01X08
- added P2: CONN_DATOS, Pin_Headers:Pin_Header_Straight_1x08, symbol CONN_01X08
- C1: footprint Capacitors_THT:C_Disc_D5.0mm_W2.5mm_P5.00mm -> Capacitors_SMD:C_1206_HandSoldering
- C2: footprint Capacitors_THT:CP_Radial_D5.0mm_P2.00mm -> Capacitors_SMD:C_1206_HandSoldering
- D1, D3: symbol LED -> LED-RESCUE-ecoBeat_3
- F1: footprint (none) -> fuse:Fuse_Horizontal_RM10mm
- J1: footprint (none) -> Connect:bornier2
- J2: footprint (none) -> Connect:bornier3
- J3: footprint (none) -> Wire_Pads:SolderWirePad_single_0-8mmDrill
- R1, R10, R2, R3, R4, R5, R6, R8, R9: footprint Resistors_THT:R_Axial_DIN0207_L6.3mm_D2.5mm_P10.16mm_Horizontal -> Resistors_SMD:R_1206
Connections:
- net labels removed: L2
- wire segments 55 -> 52
- no-connect marks 8 -> 27
Other:
- moved on the sheet: D1, D3, R6, R8, U1

Commit message: primera version para probar
Connections:
- net labels added: driver, receiver, rx_wemos, tx_wemos
- no-connect marks 27 -> 28
Other:
- moved on the sheet: J2, P1, P2, R1, R10, R2, R3, R4, R5, R9, U1, U3
