File: ecomodbus_hardware/PCB 2/modbus2.sch (KiCad schematic (older format))
At the start: 22 parts, among them J3 Test_5V, P1 CONN_VCC, P2 CONN_DATOS, P3 CONN_01X06, P4 CONN_01X01, U1 WeMos_mini, U2 ACDC-5V, U3 MAX_485

Commit message: pdb 2
Connections:
- wire segments 62 -> 60
Changed lines of the file:
@@
 EESchema Schematic File Version 2
-LIBS:ecoBeat_3-rescue
 LIBS:power
 LIBS:device
@@
 LIBS:wemos_mini
 LIBS:ecomodbus
-LIBS:ecoBeat_3-cache
 EELAYER 25 0
 EELAYER END
@@
 	0    -1   -1   0
 $EndComp
-Wire Wire Line
-	2400 1295 2400 1395
-Wire Wire Line
-	2000 1295 2000 1395
-Wire Wire Line
-	7405 4395 7505 4395
-Connection ~ 7405 4395
-Wire Wire Line
-	7955 4395 7805 4395
-Wire Wire Line
-	8255 4395 8555 4395
-Wire Wire Line
-	5810 2810 4930 2810
-Wire Wire Line
-	5715 1840 5715 1665
-Wire Wire Line
-	5430 1840 6000 1840
-Wire Wire Line
-	6000 1840 6000 2025
-Wire Wire Line
-	5810 2025 5810 1840
-Connection ~ 5810 1840
-Wire Wire Line
-	5430 1840 5430 2025
-Connection ~ 5715 1840
-Wire Wire Line
-	5620 2025 5620 1840
-Connection ~ 5620 1840
-Wire Wire Line
-	5430 2325 5430 2510
-Connection ~ 5430 2510
-Wire Wire Line
-	5620 2325 5620 2610
-Connection ~ 5620 2610
-Wire Wire Line
-	5810 2325 5810 2810
-Wire Wire Line
-	6000 2325 6000 2910
-Wire Wire Line
-	7380 2610 8740 2610
-Wire Wire Line
-	8840 2810 7380 2810
-Wire Wire Line
-	8840 2610 8840 2810
-Wire Wire Line
-	7900 2325 7900 2610
-Connection ~ 7900 2610
-Wire Wire Line
-	7900 3100 7900 2810
-Connection ~ 7900 2810
-Wire Wire Line
-	8090 2610 8090 2325
-Connection ~ 8090 2610
-Wire Wire Line
-	8090 2025 8090 1910
-Wire Wire Line
-	8090 1910 8270 1910
-Wire Wire Line
-	8270 1910 8270 2810
-Connection ~ 8270 2810
-Wire Wire Line
-	5155 4225 6130 4225
-Connection ~ 5385 4225
-Wire Wire Line
-	5155 4525 5685 4525
-Wire Wire Line
-	5155 4375 5155 4525
-Connection ~ 5385 4525
-Connection ~ 5685 4225
-Wire Wire Line
-	7900 2025 7900 1665
-Wire Wire Line
-	6980 2310 6980 2115
-Wire Wire Line
-	3930 4225 4005 4225
-Wire Wire Line
-	3935 4375 4255 4375
-Wire Wire Line
-	4205 4225 4255 4225
-Wire Wire Line
-	5385 4225 5385 4100
-Wire Wire Line
-	5620 2610 5535 2610
-Wire Wire Line
-	5535 2610 5535 2710
-Wire Wire Line
-	4930 2710 5885 2710
-Wire Wire Line
-	5430 2510 5350 2510
-Wire Wire Line
-	5350 2510 5350 2945
-Wire Wire Line
-	5350 2610 4930 2610
-Wire Wire Line
-	3120 2715 2970 2715
-Wire Wire Line
-	2790 2915 3120 2915
-Wire Wire Line
-	3120 3015 3120 3350
-Wire Wire Line
-	8255 4090 8555 4090
-Wire Wire Line
-	7805 4090 7955 4090
-Wire Wire Line
-	7505 4090 7405 4090
-Wire Wire Line
-	7405 4090 7405 4645
-Wire Wire Line
-	5385 4585 5385 4525
 $Comp
 L GND #PWR010
@@
 	1    0    0    -1
 $EndComp
-Wire Wire Line
-	1520 1400 1520 1440
-Wire Wire Line
-	9025 3010 8915 3010
-Wire Wire Line
-	9025 3110 8915 3110
 Text Label 8705 3055 0    60   ~ 0
 L_IN
 Text Label 8690 3150 0    60   ~ 0
 N_IN
-Wire Wire Line
-	6580 2510 6000 2510
-Connection ~ 6000 2510
-Wire Wire Line
-	6580 2610 5810 2610
-Connection ~ 5810 2610
-Wire Wire Line
-	6000 2910 4930 2910
-Wire Wire Line
-	6580 2810 5885 2810
-Wire Wire Line
-	5885 2810 5885 2710
-Connection ~ 5535 2710
-Wire Wire Line
-	6580 2910 6100 2910
-Wire Wire Line
-	6100 2910 6100 2945
-Wire Wire Line
-	6100 2945 5350 2945
-Connection ~ 5350 2610
 Text GLabel 8915 3010 0    60   Input ~ 0
 L_IN
@@
 L_IN
 Wire Wire Line
-	8840 2610 9025 2610
+	2400 1295 2400 1395
+Wire Wire Line
+	2000 1295 2000 1395
+Wire Wire Line
+	7405 4395 7505 4395
+Connection ~ 7405 4395
+Wire Wire Line
+	7955 4395 7805 4395
+Wire Wire Line
+	8255 4395 8555 4395
+Wire Wire Line
+	5810 2810 4930 2810
+Wire Wire Line
+	5715 1840 5715 1665
+Wire Wire Line
+	5430 1840 6000 1840
+Wire Wire Line
+	6000 1840 6000 2025
+Wire Wire Line
+	5810 2025 5810 1840
+Connection ~ 5810 1840
+Wire Wire Line
+	5430 1840 5430 2025
+Connection ~ 5715 1840
+Wire Wire Line
+	5620 2025 5620 1840
+Connection ~ 5620 1840
+Wire Wire Line
+	5430 2325 5430 2510
+Connection ~ 5430 2510
+Wire Wire Line
+	5620 2325 5620 2610
+Connection ~ 5620 2610
+Wire Wire Line
+	5810 2325 5810 2810
+Wire Wire Line
+	6000 2325 6000 2910
+Wire Wire Line
+	7380 2610 9025 2610
+Wire Wire Line
+	7380 2810 8840 2810
+Wire Wire Line
+	7900 2325 7900 2610
+Connection ~ 7900 2610
+Wire Wire Line
+	7900 3100 7900 2810
+Connection ~ 7900 2810
+Wire Wire Line
+	8090 2610 8090 2325
+Connection ~ 8090 2610
+Wire Wire Line
+	8090 2025 8090 1910
+Wire Wire Line
+	8090 1910 8270 1910
+Wire Wire Line
+	8270 1910 8270 2810
+Connection ~ 8270 2810
+Wire Wire Line
+	5155 4225 6130 4225
+Connection ~ 5385 4225
+Wire Wire Line
+	5155 4525 5685 4525
+Wire Wire Line
+	5155 4375 5155 4525
+Connection ~ 5385 4525
+Connection ~ 5685 4225
+Wire Wire Line
+	7900 2025 7900 1665
+Wire Wire Line
+	6980 2310 6980 2115
+Wire Wire Line
+	3930 4225 4005 4225
+Wire Wire Line
+	3935 4375 4255 4375
+Wire Wire Line
+	4205 4225 4255 4225
+Wire Wire Line
+	5385 4225 5385 4100
+Wire Wire Line
+	5620 2610 5535 2610
+Wire Wire Line
+	5535 2610 5535 2710
+Wire Wire Line
+	4930 2710 5885 2710
+Wire Wire Line
+	5430 2510 5350 2510
+Wire Wire Line
+	5350 2510 5350 2945
+Wire Wire Line
+	5350 2610 4930 2610
+Wire Wire Line
+	3120 2715 2970 2715
+Wire Wire Line
+	2790 2915 3120 2915
+Wire Wire Line
+	3120 3015 3120 3350
+Wire Wire Line
+	8255 4090 8555 4090
+Wire Wire Line
+	7805 4090 7955 4090
+Wire Wire Line
+	7505 4090 7405 4090
+Wire Wire Line
+	7405 4090 7405 4645
+Wire Wire Line
+	5385 4585 5385 4525
+Wire Wire Line
+	1520 1400 1520 1440
+Wire Wire Line
+	9025 3010 8915 3010
+Wire Wire Line
+	9025 3110 8915 3110
+Wire Wire Line
+	6580 2510 6000 2510
+Connection ~ 6000 2510
+Wire Wire Line
+	6580 2610 5810 2610
+Connection ~ 5810 2610
+Wire Wire Line
+	6000 2910 4930 2910
+Wire Wire Line
+	6580 2810 5885 2810
+Wire Wire Line
+	5885 2810 5885 2710
+Connection ~ 5535 2710
+Wire Wire Line
+	6580 2910 6100 2910
+Wire Wire Line
+	6100 2910 6100 2945
+Wire Wire Line
+	6100 2945 5350 2945
+Connection ~ 5350 2610
 Wire Wire Line
 	9025 2710 8740 2710
 Wire Wire Line
-	8740 2710 8740 2610
+	8840 2810 8840 2710
+Connection ~ 8840 2710
 $EndSCHEMATC
